File: esp_12_f_595/esp_12_f_595.kicad_pcb (KiCad board)
At the start: 2 copper layers, 78.7 x 29.2 mm, 21 parts, among them P0 RGB_OUT, P1 RGB_OUT, P2 RGB_OUT, P3 CONN_01X04, P4 MicroB, SW1 TACTILE, U1 74HC595, U2 74HC595, U3 AP1117v3.3, U4 74HC595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

Commit message: add first try.
Parts:
- moved R3 2.65 mm to (141.9, 86.6), turned to 180 degrees
- moved SW1 1.99 mm to (121.2, 82.5)
- moved R1 1.13 mm to (96.9, 94.2), turned to 90 degrees
Routing:
- net GND: track 0.00 -> 207.4 mm, vias 0 -> 10
- net CLK: track 0.00 -> 101.6 mm, vias 0 -> 2
- net +5V: track 0.00 -> 85.6 mm, vias 0 -> 1
- net +3V3: track 0.00 -> 84.4 mm, vias 0 -> 5
- net OEX: track 0.00 -> 80.7 mm, vias 0 -> 5
- net C: track 0.00 -> 70.6 mm
- net D: track 0.00 -> 67.4 mm
- net OE: track 0.00 -> 65.5 mm
- net STB: track 0.00 -> 64.3 mm
- net A: track 0.00 -> 64.2 mm
- net B: track 0.00 -> 63.6 mm, vias 0 -> 1
- net BCK: track 0.00 -> 62.6 mm
- net WCK: track 0.00 -> 61.6 mm, vias 0 -> 4
- net GPIO0: track 0.00 -> 46.4 mm
- net D-: track 0.00 -> 28.5 mm
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- added copper zone on B.Cu, net GND
- added copper zone on F.Cu, net GND
Other:
- net class Default: clearance 0.2286 -> 0.254
- rule trace_clearance: 0.2286 -> 0.254

Commit message: Update design
Parts:
- added H1: MH, SMTPIN, F.Cu at (153.7, 104.1)
- added H2: MH, SMTPIN, F.Cu at (71.8, 78.7)
- added H3: MH, SMTPIN, F.Cu at (153.7, 78.7)
- added H4: MH, SMTPIN, F.Cu at (71.8, 104.1)
- added P5: CONN_01X04, PHOENIX1933202, F.Cu at (137.4, 81.2)
- moved P4 0.25 mm to (114.3, 78.5)
Routing:
- net +5V: track 85.6 -> 124.0 mm, vias 1 -> 2
- net GND: track 207.4 -> 231.6 mm
- net D+: track 23.6 -> 27.0 mm
- net GPIO0: track 46.4 -> 48.3 mm
Other:
- board size 78.7 x 29.2 mm -> 85.7 x 29.2 mm
- board text added: "5V"
- board text added: "GND"

Commit message: some tweaks
Routing:
- net GND: track 231.6 -> 234.8 mm, vias 10 -> 11
- net (no net): track 2.54 -> 1.27 mm
- net Net-(U1-Pad9): track 6.61 -> 6.64 mm, vias 2 -> 0

Commit message: further tweaks
Parts:
- moved P2 0.79 mm to (138.9, 101.6)
- moved P1 0.40 mm to (112.6, 101.6)
- moved U3 0.13 mm to (104.1, 81.9)
Connections:
- net Net-(ESP1-Pad22) renamed TX
- net Net-(U1-Pad9) renamed SER1
- net Net-(U2-Pad9) renamed SER2
- net Net-(U4-Pad9) renamed SER3
- ESP1 pad 10: (no net) -> Net-(ESP1-Pad10)
- ESP1 pad 11: (no net) -> Net-(ESP1-Pad11)
- ESP1 pad 12: (no net) -> Net-(ESP1-Pad12)
- ESP1 pad 13: (no net) -> Net-(ESP1-Pad13)
- ESP1 pad 14: (no net) -> Net-(ESP1-Pad14)
- ESP1 pad 2: (no net) -> Net-(ESP1-Pad2)
- ESP1 pad 4: (no net) -> Net-(ESP1-Pad4)
- ESP1 pad 5: (no net) -> Net-(ESP1-Pad5)
- ESP1 pad 6: (no net) -> Net-(ESP1-Pad6)
- ESP1 pad 9: (no net) -> Net-(ESP1-Pad9)
- H1 pad 1: (no net) -> Net-(H1-Pad1)
- H2 pad 1: (no net) -> Net-(H2-Pad1)
- H3 pad 1: (no net) -> Net-(H3-Pad1)
- H4 pad 1: (no net) -> Net-(H4-Pad1)
- P4 pad 4: (no net) -> Net-(P4-Pad4)
- SW1 pad 2: (no net) -> Net-(SW1-Pad2)
- SW1 pad 3: (no net) -> Net-(SW1-Pad3)
- U1 pad 15: (no net) -> Net-(U1-Pad15)
- U1 pad 7: (no net) -> Net-(U1-Pad7)
- U2 pad 15: (no net) -> Net-(U2-Pad15)
- U2 pad 7: (no net) -> Net-(U2-Pad7)
- U4 pad 15: (no net) -> Net-(U4-Pad15)
- U4 pad 7: (no net) -> Net-(U4-Pad7)
- U5 pad 7: (no net) -> Net-(U5-Pad7)
- U5 pad 9: (no net) -> Net-(U5-Pad9)
Routing:
- net +5V: track 124.0 -> 113.3 mm, vias 2 -> 1
- net GND: track 234.8 -> 242.0 mm, vias 11 -> 14
- net D+: track 27.0 -> 23.7 mm
- net B0_0: track 27.1 -> 29.7 mm
- net +3V3: track 84.4 -> 86.1 mm, vias 5 -> 3
- net GPIO0: track 48.3 -> 46.8 mm
- net (no net): track 1.27 -> 0.00 mm, vias 2 -> 0
- net CLK: track 101.6 -> 100.7 mm
- net WCK: track 61.6 -> 60.7 mm, vias 4 -> 5
- net B: track 63.6 -> 62.8 mm
- net OE: track 65.5 -> 64.8 mm
- net A: track 64.2 -> 63.6 mm
Other:
- net class Default: trace_width 0.2794 -> 0.3302
